File: esp32_breakout.kicad_sch (KiCad schematic)
At the start: 17 parts, among them J4 USB_C_Receptacle_USB2.0_16P, SW1 USAKRO UK-B0227-G4.3-B-250, SW2 USAKRO UK-B0227-G4.3-B-250, U7 ESP32-S3-WROOM-1U

Commit message: remove remainder of leftofer schematics
Parts:
- removed C22: 22uF, Capacitor_SMD:C_0805_2012Metric, symbol Device:C_Small
- removed C23, C25: 0.1μF, Capacitor_SMD:C_0402_1005Metric, symbol Device:C_Small
- removed C24: 1uF, Capacitor_SMD:C_0603_1608Metric, symbol Device:C_Small
- removed D8: LED-Y, LED_SMD:LED_0805_2012Metric, symbol Device:LED
- removed R29: 10k, Resistor_SMD:R_0402_1005Metric, symbol Device:R_Small_US
- removed R30: 1k, Resistor_SMD:R_0402_1005Metric, symbol Device:R_Small_US
- removed R33: 270k, Resistor_SMD:R_0402_1005Metric, symbol Device:R_Small_US
- removed R34: 39k, Resistor_SMD:R_0402_1005Metric, symbol Device:R_Small_US
- removed SW1, SW2: USAKRO UK-B0227-G4.3-B-250, Button_Switch_SMD:SW_Tactile_SPST_NO_Straight_CK_PTS636Sx25SMTRLFS, symbol Switch:SW_Push
- removed U7: ESP32-S3-WROOM-1U, RF_Module:ESP32-S3-WROOM-1U, symbol RF_Module:ESP32-S3-WROOM-1
- C26: value 0.1μF -> 100nF; footprint Capacitor_SMD:C_0402_1005Metric -> (none); LCSC C307331 -> (none); MPN CL05B104KO5NNNC -> (none)
- R31, R32: footprint Resistor_SMD:R_0402_1005Metric -> (none)
Connections:
- no-connect marks 16 -> 2
Other:
- note removed: "24V*(39/(39+270))=3.03V SAFE_DETECT"
- note removed: "24V_Safe detect"
- note removed: "Wifi Indicator"
- moved on the sheet: C26, CR1, J4, R31, R32
