File: panda.kicad_pcb (KiCad board)
At the start: 4 copper layers, 100 x 130 mm, 270 parts, among them J1 Conn_01x02, J10 Conn_01x02, J11 4-Pin Load Cell, J12 5-Pin Load Cell, J13 Conn_02x01, J14 Conn_01x02, J15 Conn_01x02, J16 Conn_01x02, J17 Conn_01x02, J18 Conn_01x02, J19 Conn_01x02, J2 Conn_02x01, J20 395934308, J3 Conn_02x01, J4 USB_C_Receptacle_USB2.0_16P, J5 Conn_01x02, J6 Conn_01x02, J7 Conn_01x02, J8 Conn_01x02, J9 Conn_01x02, K1 G5Q-1A DC24, K2 G5Q-1 DC24, K3 G5Q-1 DC24, Q1 BSS138, Q10 BSS138, Q11 BSS138, Q12 BSS138, Q2 BSS138, Q3 DMP6023LE-13, Q4 BSS138, Q5 BSS138, Q6 BSS138, Q7 BSS138, Q8 BSS138, Q9 BSS138, SW1 USAKRO UK-B0227-G4.3-B-250, SW2 USAKRO UK-B0227-G4.3-B-250, U1 LM3880-1AA, U10 ADS112C04, U11 ADS112C04, U12 INA187A2, U13 ADS112C04, U2 LMR33630BDDA, U3 TPS78533QKVURQ1, U4 TLC555xPS, U5 TPS78450QDBVRQ1, U6 LM66200DRLR, U7 ESP32-S3-WROOM-1U, U8 ADS112C04, U9 ADS112C04

Commit message: clean up repo
Parts:
- removed BZ1: YS-SBZ9650DYB05, Library:YS-SBZ9650DYB05
- removed C1, C14, C15, C18, C19, C21, C23, C25, C26, C27, C28, C33, C34, C39, C40, C42, C45, C47, C48, C50, C53, C61, C62, C63, C7: 0.1μF, Capacitor_SMD:C_0402_1005Metric
- removed C10, C12, C22: 22uF, Capacitor_SMD:C_0805_2012Metric
- removed C11: 10nF, Capacitor_SMD:C_0402_1005Metric
- removed C13, C17, C20, C8: 10uF, Capacitor_SMD:C_0805_2012Metric
- removed C16: 2.2uF, Capacitor_SMD:C_0603_1608Metric
- removed C2: 100uF, Capacitor_SMD:CP_Elec_10x10
- removed C24, C6: 1uF, Capacitor_SMD:C_0603_1608Metric
- removed C29, C30, C31, C32, C35, C36, C37, C38, C64, C65, C66, C67: 150nF, Capacitor_SMD:C_0402_1005Metric
- removed C3: 10uF, Capacitor_SMD:C_1812_4532Metric
- removed C4: 10uF, Capacitor_SMD:C_1206_3216Metric
- removed C41, C43, C44, C46, C49, C51, C52, C54: 10nF, Capacitor_SMD:C_0603_1608Metric
- removed C5: 220nF, Capacitor_SMD:C_0805_2012Metric
- removed C55, C56, C57, C58, C59, C60: 3.3uF, Capacitor_SMD:C_0805_2012Metric
- removed C9: 3pF, Capacitor_SMD:C_0603_1608Metric
- removed CR1: USBLC6-2SC6, Package_TO_SOT_SMD:SOT-23-6
- removed D1, D25, D3, D4, D6, D7: LED-G, LED_SMD:LED_0805_2012Metric
- removed D10, D11, D12, D13, D14, D15, D16, D34, D35, D36, D37, D9: BAT54SW, Package_TO_SOT_SMD:SOT-323_SC-70
- removed D17, D18, D19, D20, D21, D22, D23, D24: BAV199, Package_TO_SOT_SMD:SOT-23
- removed D2: SMCJ26A-13-F, Diode_SMD:D_SMC
- removed D26, D27, D28, D29, D30, D31, D32, D33, D38, D5: SK44BL, Diode_SMD:D_SMB
- removed D8: LED-Y, LED_SMD:LED_0805_2012Metric
- removed F1, F2: Fuse, Fuse:Fuseholder_Blade_Mini_Keystone_3568
- removed G*** (x2): LOGO, LOGO
- removed H1, H2, H3, H4: MountingHole_Pad, MountingHole:MountingHole_3.2mm_M3_ISO7380_Pad
- removed J1, J10, J14, J15, J16, J17, J18, J19, J5, J6, J7, J8, J9: Conn_01x02, Connector_Molex:Molex_Micro-Fit_3.0_43650-0215_1x02_P3.00mm_Vertical
- removed J11: 4-Pin Load Cell, Connector_Molex:Molex_Micro-Fit_3.0_43650-0415_1x04_P3.00mm_Vertical
- removed J12: 5-Pin Load Cell, Connector_Molex:Molex_Micro-Fit_3.0_43650-0515_1x05_P3.00mm_Vertical
- removed J13, J2, J3: Conn_02x01, Connector_Molex:Molex_Mini-Fit_Jr_5566-02A_2x01_P4.20mm_Vertical
- removed J20: 395934308, Library:CONN_SD-39543-002_NONE_08P_MOL
- removed J4: USB_C_Receptacle_USB2.0_16P, Connector_USB:USB_C_Receptacle_G-Switch_GT-USB-7051x
- removed K1: G5Q-1A DC24, Relay_THT:Relay_SPST_Omron-G5Q-1A
- removed K2, K3: G5Q-1 DC24, Relay_THT:Relay_SPDT_Omron-G5Q-1
- removed L1: 4.7uH, Inductor_SMD:L_Bourns_SRP7028A_7.3x6.6mm
- removed Q1, Q10, Q11, Q12, Q2, Q4, Q5, Q6, Q7, Q8, Q9: BSS138, Package_TO_SOT_SMD:SOT-23-3
- removed Q3: DMP6023LE-13, Package_TO_SOT_SMD:SOT-223-3_TabPin2
- removed R1, R2, R28, R3, R4, R5: 3.3k, Resistor_SMD:R_0402_1005Metric
- removed R10, R12, R14, R20, R21, R23, R8, R83, R84, R87, R88, R91, R92: 100k, Resistor_SMD:R_0603_1608Metric
- removed R11, R13, R34, R76, R9: 39k, Resistor_SMD:R_0402_1005Metric
- removed R15, R18, R19, R27, R29, R39, R44, R53, R62, R77, R78, R97, R98: 10k, Resistor_SMD:R_0402_1005Metric
- removed R16, R79, R80, R81, R82, R85, R86, R89, R90: 100, Resistor_SMD:R_0402_1005Metric
- removed R17: 470k, Resistor_SMD:R_0603_1608Metric
- removed R22: 23.2k, Resistor_SMD:R_0603_1608Metric
- removed R24: 18k, Resistor_SMD:R_0603_1608Metric
- removed R25: 1.2k, Resistor_SMD:R_0402_1005Metric
- removed R26: 160k, Resistor_SMD:R_0402_1005Metric
- removed R30, R35, R36, R37, R38, R40, R41, R42, R43, R49, R50, R51, R52, R58, R59, R6, R60, R61, R7, R94, R95, R96: 1k, Resistor_SMD:R_0402_1005Metric
- removed R31, R32: 5.1k, Resistor_SMD:R_0402_1005Metric
- removed R33: 270k, Resistor_SMD:R_0402_1005Metric
- removed R45, R46, R47, R48, R54, R55, R56, R57: 1M, Resistor_SMD:R_0402_1005Metric
- removed R63, R64, R67, R68, R71, R72: 10, Resistor_SMD:R_0402_1005Metric
- removed R65, R66, R69, R70, R73, R74: 250, Resistor_SMD:R_0603_1608Metric
- removed R75: 10m 1W, Resistor_SMD:R_1206_3216Metric
- removed R93: 47, Resistor_SMD:R_0402_1005Metric
- removed R99: 2.2k, Resistor_SMD:R_0402_1005Metric
- removed SW1, SW2: USAKRO UK-B0227-G4.3-B-250, Button_Switch_SMD:SW_Tactile_SPST_NO_Straight_CK_PTS636Sx25SMTRLFS
- removed TP1: TestPoint, TestPoint:TestPoint_Loop_D2.50mm_Drill1.0mm
- removed TP2: SDA, TestPoint:TestPoint_Pad_D1.5mm
- removed TP3: SCL, TestPoint:TestPoint_Pad_D1.5mm
- removed TP4: TP_+3.3V, TestPoint:TestPoint_Pad_D1.0mm
- removed TP5: TP_+5V, TestPoint:TestPoint_Pad_D1.0mm
- removed U1: LM3880-1AA, Package_TO_SOT_SMD:SOT-23-6
- removed U10, U11, U13, U8, U9: ADS112C04, Package_SO:TSSOP-16_4.4x5mm_P0.65mm
- removed U12: INA187A2, Package_TO_SOT_SMD:SOT-23-6
- removed U2: LMR33630BDDA, Package_SO:Texas_HSOP-8-1EP_3.9x4.9mm_P1.27mm_ThermalVias
- removed U3: TPS78533QKVURQ1, Package_TO_SOT_SMD:TO-252-4
- removed U4: TLC555xPS, Package_SO:VSSOP-8_3x3mm_P0.65mm
- removed U5: TPS78450QDBVRQ1, Package_TO_SOT_SMD:SOT-23-5
- removed U6: LM66200DRLR, Package_TO_SOT_SMD:SOT-583-8
- removed U7: ESP32-S3-WROOM-1U, RF_Module:ESP32-S3-WROOM-1U
Routing:
- net +24V: track 251.5 -> 0.00 mm, vias 4 -> 0
- net +5V: track 250.0 -> 0.00 mm, vias 37 -> 0
- net GND: track 208.7 -> 0.00 mm, vias 366 -> 0
- net +24V_SAFE: track 174.0 -> 0.00 mm, vias 1 -> 0
- net +3.3V: track 135.1 -> 0.00 mm, vias 14 -> 0
- net IGN_RESIST_READ: track 111.1 -> 0.00 mm, vias 2 -> 0
- net IGN_CURRENT_READ: track 107.6 -> 0.00 mm, vias 4 -> 0
- net /Power Regulation/+5.3V: track 91.1 -> 0.00 mm, vias 4 -> 0
- net I2C_SDA: track 79.6 -> 0.00 mm
- net +24V_PT: track 74.4 -> 0.00 mm, vias 7 -> 0
- net I2C_SCL: track 73.6 -> 0.00 mm
- net /Power Regulation/+24V_POST_LCKT: track 66.0 -> 0.00 mm, vias 1 -> 0
- net IGNITOR_PRIME_CTL: track 62.4 -> 0.00 mm
- net /ESP32 Breakout/USB_N: track 57.5 -> 0.00 mm
- net /ESP32 Breakout/USB_P: track 57.5 -> 0.00 mm
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- removed copper zone on F.Cu, net +24V
- removed copper zone on B.Cu, net +3.3V
- removed copper zone on B.Cu, net +5V
- removed copper zone on F.Cu, net /Ignitor Control/IGNITOR_+VE
- removed copper zone on F.Cu, net /Ignitor Control/IGN_SUPPLY
- removed copper zone on F.Cu, net /Power Regulation/+5.3V
- removed copper zone on B.Cu, net /Power Regulation/PWR_SQ
- removed copper zone on F.Cu, net /Power Regulation/SW
- removed copper zone on B.Cu, net GND
- removed copper zone on F.Cu, net GND
- removed copper zone on In1.Cu, net GND
- removed copper zone on In2.Cu, net GND
- removed copper zone on F.Cu, net Net-(J2-Pin_1)
- removed copper zone on F.Cu, net Net-(U2-FB)
Other:
- board outline removed
- board text removed: "24VIN"
- board text removed: "24V_SAFE_LOCK"
- board text removed: "AV3"
- board text removed: "AV4"
- board text removed: "AV5"
- board text removed: "AV6"
- board text removed: "AV_FILL"
- board text removed: "AV_RUN"
- board text removed: "IGNITOR"
- board text removed: "LC_FILL"
- board text removed: "LC_THRUST"
- board text removed: "PANDA Propulsion Actuation and Nominal Data Acquisition V3.0.0 Dec 21 2025 Nathan Belza"
- board text removed: "PT1"
- board text removed: "PT2"
- board text removed: "PT3"
- board text removed: "PT4"
- board text removed: "PT5"
- board text removed: "PT6"
- board text removed: "PWR_ON_SW"
- board text removed: "TC1- TC1+"
- board text removed: "TC2- TC2+"
- board text removed: "TC3- TC3+"
- board text removed: "TC4- TC4+"
- board text removed: "https://github.com/Queens-Rocket-Engineering-Team/prop-panda Based on PANDA Design Spec Rev 1."
